File: Hardware/1.EnvironmentSensors/Kicad/EnvironmentSensors.kicad_pcb (KiCad board)
At the start: 2 copper layers, 60 x 60 mm, 18 parts, among them J1 Conn_01x10_Pin, J2 Conn_01x10_Pin, U1 SHT4x, U2 BME680, U3 LPS22HB

Commit message: Update layout with changes made in schematic
Parts:
- added C5: 100n, Capacitor_SMD:C_0603_1608Metric, F.Cu at (138.9, 85.5)
- added C6: 100n, Capacitor_SMD:C_0603_1608Metric, F.Cu at (121.1, 90.5)
- C3, C4: footprint Capacitor_SMD:C_0402_1005Metric -> Capacitor_SMD:C_0603_1608Metric
- R1, R2, R3, R4: footprint Resistor_SMD:R_0402_1005Metric -> Resistor_SMD:R_0603_1608Metric
- moved JP3 4.74 mm to (134.4, 95.5), turned to -90 degrees
- moved C2 4.16 mm to (135.3, 72.7), turned to 0 degrees
- moved REF** 2.44 mm to (123.2, 80.0)
- moved C1 1.57 mm to (132.6, 75.5), turned to 90 degrees
- moved R3 1.00 mm to (133.3, 87.5)
- moved C4 0.94 mm to (145.0, 87.5), turned to 0 degrees
- moved R4 0.92 mm to (141.9, 93.2)
- moved U2 0.85 mm to (135.3, 75.5)
- moved C3 0.84 mm to (146.9, 90.8)
- moved R2 0.58 mm to (137.3, 87.5)
- moved R1 0.38 mm to (133.3, 85.5)
Routing:
- net EXT_3V3: track 30.1 -> 20.3 mm
- net GND: track 19.1 -> 26.9 mm, vias 2 -> 4
- net Net-(JP2-B): track 14.2 -> 19.3 mm
- net +3.3V: track 37.8 -> 42.4 mm, vias 6 -> 8
- net Net-(JP1-B): track 26.2 -> 22.3 mm
- net I2C_SDA: track 47.9 -> 50.2 mm
